Commit message: added transmissions

File: starship/urdf/starship.urdf (robot description, URDF)
Before this commit: robot starship, 5 links, 4 joints
Joints:
- joint Joint_Arm_L: limit lower=-1.57 upper=1.57 effort=0 velocity=0 -> lower=-1.57 upper=1.57
- joint Joint_Arm_R: limit lower=-1.57 upper=1.57 effort=0 velocity=0 -> lower=-1.57 upper=1.57
- joint Joint_Leg_L: limit lower=-1.57 upper=1.57 effort=0 velocity=0 -> lower=-1.57 upper=1.57
- joint Joint_Leg_R: limit lower=-1.57 upper=1.57 effort=0 velocity=0 -> lower=-1.57 upper=1.57
